File: IOB-Adapter-Turtle.sch (EAGLE design)
At the start: 5 parts

Commit message: silkscreen tweeks
Parts:
- added C1, C2, C3: 0.01uF, SPCoast:CAP0603
- added D1, D2, D3: BAT54S, SPCoast:DIODE-BAT54S23
- added D4: 4.7v, SPCoast:DIODESOT23
- added R5, R6, RM: 1K0, SPCoast:R0603-RES
- added RN, RO, RR: 82R, SPCoast:R0805-RES
- R1, R2, R3: value NOSTUFF -> 10k; device SPCoast:RPTH-R0 -> SPCoast:R0805-RES
- R4: value NOSTUFF -> 1K0; device SPCoast:RPTH-R0 -> SPCoast:R0603-RES
Connections:
- removed net N$1: JP1.1, R1.1
- removed net N$4: JP1.9, R4.1
- new net IO1: JP1.1, RR.2
- new net IO2: JP1.3, RN.2
- new net IO3: JP1.7, RO.2
- new net IO4: JP1.9, RM.1
- new net N$14: C3.1, D3.COM, R6.2, RO.1
- net GND: now also C1.2, C2.2, C3.2, D1.A1, D2.A1, D3.A1, D4.A
- net N$2: now also C2.1, D2.COM, R5.2, RN.1; no longer JP1.3, R2.1
- net N$3: now also C1.1, D1.COM, R4.2, RR.1; no longer JP1.7, R3.1
- net P1: now also R4.1
- net P2: now also R5.1
- net P3: now also R6.1
- net P4: now also D4.C, RM.2; no longer R4.2
- net VCC: now also D1.C2, D2.C2, D3.C2, R1.1, R2.1, R3.1
Other:
- note added: "!Motor Control"
- note added: "!Normal Feedback"
- note added: "!Occupied Feedback"
- note added: "!Reverse Feedback"
- note added: "3.0"
- note added: "3.0: Added low pass filter to feedback inputs"
- note added: "IO4 Turtle interface"
- note added: "Turtle - Tortoise Interface"
- note removed: "Generic I/O"
